Commit message: Working with Gazebo

File: kurtana_bringup/urdf/kinect.urdf.xacro (robot description, xacro)
@@ -1,10 +1,7 @@
 <?xml version="1.0"?>
-<robot xmlns:sensor="http://playerstage.sourceforge.net/gazebo/xmlschema/#sensor"
-  xmlns:controller="http://playerstage.sourceforge.net/gazebo/xmlschema/#controller"
-  xmlns:interface="http://playerstage.sourceforge.net/gazebo/xmlschema/#interface"
+<robot
   xmlns:xacro="http://ros.org/wiki/xacro"
   name="${camera}">
   <include filename="$(find kurtana_bringup)/urdf/common.xacro" />
-  <include filename="$(find kurtana_bringup)/urdf/openni.gazebo.xacro" />
   <xacro:macro name="kinect" params="camera">
     <link name="${camera}_link">
@@ -50,6 +47,4 @@
       </inertial>
     </link>
-    <!-- OpenNI IR sensor Gazebo extensions -->
-    <xacro:openni_ir_gazebo_v0 link_name="${camera}_depth_frame" frame_name="${camera}_depth_optical_frame" camera_name="${camera}" />
     <joint name="${camera}_rgb_joint" type="fixed">
       <origin xyz="0 -0.005 0" rpy="0 0 0" />
@@ -79,6 +74,4 @@
       </inertial>
     </link>
-    <!-- OpenNI RGB sensor Gazebo extensions -->
-    <xacro:openni_rgb_gazebo_v0 link_name="${camera}_rgb_frame" frame_name="${camera}_rgb_optical_frame" camera_name="${camera}" />
   </xacro:macro>
 </robot>

File: kurtana_bringup/urdf/kurtana.urdf.xacro (robot description, xacro)
@@ -4,9 +4,33 @@
   name="kurtana">
   <xacro:property name="top_y_offset" value="0.00" />
-  <xacro:property name="base_z_offset" value="0.20" /> <!-- distance from base_link to top of cover surface -->
-  <include filename="$(find p2os_urdf)/defs/pioneer3dx.xacro" />
+  <xacro:property name="base_z_offset" value="0.60" /> <!-- distance from base_link to top of cover surface -->
   <include filename="$(find kurtana_bringup)/urdf/kurtana_top.urdf.xacro" />
-  <joint name="top_base_joint" type="fixed">
-    <parent link="top_plate" />
+	<link name="base_link">
+		<visual name="base_visual">
+			<origin xyz="-0.045 0 0.148" rpy="0 0 0"/>
+			<geometry name="pioneer_geom">
+				<mesh filename="package://p2os_urdf/meshes/p3dx_meshes/chassis.stl"/>
+			</geometry>
+			<material name="ChassisRed">
+				<color rgba="0.851 0.0 0.0 1.0"/>
+			</material>
+		</visual>
+    <inertial>
+			<mass value="500" />
+			<inertia ixx="500"  ixy="0"  ixz="0" iyy="500" iyz="0" izz="500" />
+			<origin/>
+		</inertial>
+	<collision>
+			<origin xyz="-0.045 0 0.148" rpy="0 0 0"/>
+			<geometry name="pioneer_geom">
+				<mesh filename="package://p2os_urdf/meshes/p3dx_meshes/chassis.stl"/>
+			</geometry>
+	</collision>
+	</link>
+	<gazebo reference="base_link">
+		<material value="Gazebo/Red"/>
+	</gazebo>
+  <joint name="base_joint" type="fixed">
+    <parent link="base_link" />
     <child link="kurtana_baseplate_link" />
     <origin xyz="0 ${top_y_offset} ${base_z_offset + rackplate_height/2}" />

File: kurtana_bringup/urdf/kurtana_rack.urdf.xacro (robot description, xacro)
@@ -3,7 +3,5 @@
   <!-- *** TODO: roll should be yaw here *** -->
   <!-- ******************** -->
-<robot xmlns:sensor="http://playerstage.sourceforge.net/gazebo/xmlschema/#sensor"
-  xmlns:controller="http://playerstage.sourceforge.net/gazebo/xmlschema/#controller"
-  xmlns:interface="http://playerstage.sourceforge.net/gazebo/xmlschema/#interface"
+<robot
   xmlns:xacro="http://ros.org/wiki/xacro"
   name="kurtana_rack">
@@ -268,19 +266,4 @@
     <xacro:box_inertial x="${kinect_mounting_plate_length}" y="${kinect_mounting_plate_width}" z="${kinect_mounting_plate_height}" mass="${kinect_mounting_plate_mass}" />
   </link>
-  <!-- ******************** -->
-  <!-- *** Gazebo stuff *** -->
-  <!-- ******************** -->
-  <!-- transmissions are required by the controller manager (here: for simulation in gazebo) -->
-  <xacro:macro name="kurtana_pole_transmission" params="name">
-    <transmission name="${name}_trans" type="pr2_mechanism_model/SimpleTransmission">
-      <actuator name="${name}_motor" />
-      <joint name="${name}_joint" />
-      <mechanicalReduction>1</mechanicalReduction>
-      <motorTorqueConstant>1</motorTorqueConstant>
-    </transmission>
-  </xacro:macro>
-  <xacro:kurtana_pole_transmission name="kurtana_stretch" />
-  <xacro:kurtana_pole_transmission name="kurtana_roll" />
-  <xacro:kurtana_pole_transmission name="kurtana_pitch" />
   <gazebo reference="kurtana_rackplate_link">
     <material value="PR2/Grey" />

File: kurtana_bringup/urdf/kurtana_top.urdf.xacro (robot description, xacro)
@@ -1,7 +1,4 @@
 <?xml version="1.0"?>
-<robot xmlns:sensor="http://playerstage.sourceforge.net/gazebo/xmlschema/#sensor"
-  xmlns:controller="http://playerstage.sourceforge.net/gazebo/xmlschema/#controller"
-  xmlns:interface="http://playerstage.sourceforge.net/gazebo/xmlschema/#interface"
-  xmlns:xacro="http://ros.org/wiki/xacro"
+<robot xmlns:xacro="http://ros.org/wiki/xacro"
   name="kurtana">
   <property name="M_PI" value="3.1415926535897931" />
@@ -24,18 +21,11 @@
   </joint>
   <!-- **************************** -->
-  <!-- *** Neuronics Katana Arm *** -->
+  <!-- *** Jaco Arm *** -->
   <!-- **************************** -->
- <include filename="$(find katana_description)/urdf/katana_300_6m180.urdf.xacro" />
+ <include filename="$(find jaco_description)/urdf/gazebo/jaco.urdf.xacro" />
   <joint name="kurtana_baseplate_katana_baseplate_joint" type="fixed">
     <parent link="katana_baseplate_link" />
-    <child link="katana_base_link" />
+    <child link="jaco_base_link" />
     <origin xyz="0 0 0" rpy="0 0 0" />
   </joint>
-  <!-- pattern for Kinect calibration -->
-   <link name="katana_pattern"></link>
-  <joint name="katana_pattern_joint" type="fixed">
-    <parent link="katana_motor4_lift_link"/>
-    <child  link="katana_pattern" />
-    <origin xyz=".075 -.035 0.00" rpy="1.571 -1.571 0.151"/>
-  </joint>
 </robot>
