Commit message: jaco base mounted horizontally

File: kurtana_bringup/urdf/kurtana_top.urdf.xacro (robot description, xacro)
@@ -27,5 +27,5 @@
     <parent link="katana_baseplate_link" />
     <child link="jaco_base_link" />
-    <origin xyz="0 0 0" rpy="0 0 0" />
+    <origin xyz="-0.27 0 0.27" rpy="${M_PI/2} ${M_PI} ${M_PI/2}" />
   </joint>
 </robot>
